Commit message: use the new urdf of quad, stop use the go1

File: source/multi_loco/multi_loco/assets/resources/urdf/braver_quad.urdf (robot description, URDF)
Before this commit: robot go1_pointfoot_quadruped, 27 links, 26 joints
Links:
- removed link base
- link trunk: geometry collision box size=0.3762 0.18 0.15; visual box size=0.3762 0.18 0.15
Joints:
- removed joint floating_base
- joint FL_abad_joint: origin xyz=0.1881 0.04675 0 -> xyz=0.1881 0.09 0
- joint FR_abad_joint: origin xyz=0.1881 -0.04675 0 -> xyz=0.1881 -0.09 0
- joint RL_abad_joint: origin xyz=-0.1881 0.04675 0 -> xyz=-0.1881 0.09 0
- joint RR_abad_joint: origin xyz=-0.1881 -0.04675 0 -> xyz=-0.1881 -0.09 0
