Commit message: modify the three forms to the code

File: source/multi_loco/multi_loco/assets/resources/urdf/braver_biped.urdf (robot description, URDF)
Before this commit: robot point_foot, 13 links, 12 joints
Links:
- link base_Link: mass 5.6 -> 3.6

File: source/multi_loco/multi_loco/assets/resources/urdf/braver_hexapod.urdf (robot description, URDF)
Before this commit: robot go1_pointfoot_quadruped, 38 links, 37 joints
Links:
- link trunk: mass 7.2 -> 10.8; geometry collision box size=0.75 0.18 0.15; visual box size=0.75 0.18 0.15
Joints:
- joint FL_abad_joint: origin xyz=0.28215 0.09 0 -> xyz=0.375 0.09 0
- joint FR_abad_joint: origin xyz=0.28215 -0.09 0 -> xyz=0.375 -0.09 0
- joint RL_abad_joint: origin xyz=-0.28215 0.09 0 -> xyz=-0.375 0.09 0
- joint RR_abad_joint: origin xyz=-0.28215 -0.09 0 -> xyz=-0.375 -0.09 0

File: source/multi_loco/multi_loco/assets/resources/urdf/braver_quad.urdf (robot description, URDF)
Before this commit: robot go1_pointfoot_quadruped, 26 links, 25 joints
Links:
- link trunk: mass 4.8 -> 7.2; geometry collision box size=0.50 0.18 0.15; visual box size=0.50 0.18 0.15
Joints:
- joint FL_abad_joint: origin xyz=0.1881 0.09 0 -> xyz=0.25 0.09 0
- joint FR_abad_joint: origin xyz=0.1881 -0.09 0 -> xyz=0.25 -0.09 0
- joint RL_abad_joint: origin xyz=-0.1881 0.09 0 -> xyz=-0.25 0.09 0
- joint RR_abad_joint: origin xyz=-0.1881 -0.09 0 -> xyz=-0.25 -0.09 0
