Commit message: more random, einsum->matmul, use the export in runner which has GNN

File: source/multi_loco/multi_loco/assets/resources/urdf/braver_hexapod.urdf (robot description, URDF)
Before this commit: robot go1_pointfoot_quadruped, 38 links, 37 joints
Links:
- link trunk: geometry collision box size=0.75 0.18 0.08; visual box size=0.75 0.18 0.15

File: source/multi_loco/multi_loco/assets/resources/urdf/braver_quad.urdf (robot description, URDF)
Before this commit: robot go1_pointfoot_quadruped, 26 links, 25 joints
Links:
- link trunk: geometry collision box size=0.50 0.18 0.08; visual box size=0.50 0.18 0.15
